Commit message: 完全没问题了

File: src/ackermann_car/urdf/ackermann_car.xacro (robot description, xacro)
@@ -1,44 +1,293 @@
 <?xml version="1.0"?>
-<robot name="ackermann_car" xmlns:xacro="http://ros.org/wiki/xacro">
-  <!-- base -->
-  <link name="base_link">
-    <visual>
-      <geometry>
-        <box size="0.6 0.3 0.1"/>
-      </geometry>
-      <origin xyz="0 0 0.05"/>
-      <material name="blue"/>
-    </visual>
-    <collision>
-      <geometry>
-        <box size="0.6 0.3 0.1"/>
-      </geometry>
-      <origin xyz="0 0 0.05"/>
-    </collision>
-    <inertial>
-      <mass value="5.0"/>
-      <inertia ixx="0.1" ixy="0" ixz="0" iyy="0.1" iyz="0" izz="0.1"/>
-    </inertial>
-  </link>
-  <xacro:macro name="wheel" params="name x y">
-    <link name="${name}">
+<robot name="ackermann_car" xmlns:xacro="http://www.ros.org/wiki/xacro">
+  <!-- 宏定义：车辆参数 -->
+  <xacro:property name="chassis_length" value="1.8"/>
+  <xacro:property name="chassis_width" value="0.8"/>
+  <xacro:property name="chassis_height" value="0.4"/>
+  <xacro:property name="wheel_radius" value="0.15"/>
+  <xacro:property name="wheel_width" value="0.1"/>
+  <xacro:property name="wheelbase" value="1.2"/>
+  <xacro:property name="track_width" value="0.6"/>
+  <xacro:property name="chassis_mass" value="50.0"/>
+  <xacro:property name="wheel_mass" value="2.0"/>
+  <!-- 宏定义：传感器参数 -->
+  <xacro:property name="lidar_height" value="0.1"/>
+  <xacro:property name="lidar_radius" value="0.05"/>
+  <xacro:property name="camera_width" value="0.1"/>
+  <xacro:property name="camera_height" value="0.05"/>
+  <xacro:property name="camera_depth" value="0.05"/>
+  <xacro:property name="imu_size" value="0.05"/>
+  <!-- 车身链接 -->
+  <link name="chassis">
+    <inertial>
+      <mass value="${chassis_mass}"/>
+      <inertia>
+        <ixx>${chassis_mass * (chassis_height*chassis_height + chassis_width*chassis_width) / 12}</ixx>
+        <iyy>${chassis_mass * (chassis_length*chassis_length + chassis_height*chassis_height) / 12}</iyy>
+        <izz>${chassis_mass * (chassis_length*chassis_length + chassis_width*chassis_width) / 12}</izz>
+        <ixy>0.0</ixy>
+        <ixz>0.0</ixz>
+        <iyz>0.0</iyz>
+      </inertia>
+    </inertial>
+    <visual>
+      <origin xyz="0 0 ${chassis_height/2}" rpy="0 0 0"/>
+      <geometry>
+        <box size="${chassis_length} ${chassis_width} ${chassis_height}"/>
+      </geometry>
+      <material name="blue">
+        <color rgba="0 0 1 1"/>
+      </material>
+    </visual>
+    <collision>
+      <origin xyz="0 0 ${chassis_height/2}" rpy="0 0 0"/>
+      <geometry>
+        <box size="${chassis_length} ${chassis_width} ${chassis_height}"/>
+      </geometry>
+    </collision>
+  </link>
+  <!-- 轮子宏 -->
+  <xacro:macro name="wheel" params="name side prefix x_offset y_offset">
+    <link name="${prefix}_${name}_wheel">
+      <inertial>
+        <mass value="${wheel_mass}"/>
+        <inertia>
+          <ixx>${wheel_mass * wheel_radius*wheel_radius / 2}</ixx>
+          <iyy>${wheel_mass * (3*wheel_radius*wheel_radius + wheel_width*wheel_width) / 12}</iyy>
+          <izz>${wheel_mass * (3*wheel_radius*wheel_radius + wheel_width*wheel_width) / 12}</izz>
+          <ixy>0.0</ixy>
+          <ixz>0.0</ixz>
+          <iyz>0.0</iyz>
+        </inertia>
+      </inertial>
       <visual>
+        <origin xyz="0 0 0" rpy="${pi/2} 0 0"/>
         <geometry>
-          <cylinder radius="0.05" length="0.02"/>
+          <cylinder radius="${wheel_radius}" length="${wheel_width}"/>
         </geometry>
-        <origin xyz="${x} ${y} 0.025" rpy="1.57 0 0"/>
-        <material name="black"/>
+        <material name="black">
+          <color rgba="0 0 0 1"/>
+        </material>
       </visual>
+      <collision>
+        <origin xyz="0 0 0" rpy="${pi/2} 0 0"/>
+        <geometry>
+          <cylinder radius="${wheel_radius}" length="${wheel_width}"/>
+        </geometry>
+      </collision>
     </link>
-    <joint name="${name}_joint" type="continuous">
-      <parent link="base_link"/>
-      <child link="${name}"/>
-      <origin xyz="${x} ${y} 0.025"/>
+    <joint name="${prefix}_${name}_wheel_joint" type="continuous">
+      <parent link="chassis"/>
+      <child link="${prefix}_${name}_wheel"/>
+      <origin xyz="${x_offset} ${y_offset * track_width/2} ${wheel_radius}" rpy="0 0 0"/>
       <axis xyz="0 1 0"/>
     </joint>
+    <xacro:if value="${prefix == 'front'}">
+      <joint name="${prefix}_${name}_steering_joint" type="revolute">
+        <parent link="chassis"/>
+        <child link="${prefix}_${name}_wheel"/>
+        <origin xyz="${x_offset} ${y_offset * track_width/2} ${wheel_radius}" rpy="0 0 0"/>
+        <axis xyz="0 0 1"/>
+        <limit lower="${-pi/4}" upper="${pi/4}" effort="100" velocity="10"/>
+      </joint>
+    </xacro:if>
   </xacro:macro>
-  <xacro:wheel name="front_left_wheel"  x="0.2"  y="0.15"/>
-  <xacro:wheel name="front_right_wheel" x="0.2"  y="-0.15"/>
-  <xacro:wheel name="rear_left_wheel"   x="-0.2" y="0.15"/>
-  <xacro:wheel name="rear_right_wheel"  x="-0.2" y="-0.15"/>
+  <!-- 定义四个轮子 -->
+  <xacro:wheel name="left" side="1" prefix="front" x_offset="${wheelbase/2}" y_offset="1"/>
+  <xacro:wheel name="right" side="-1" prefix="front" x_offset="${wheelbase/2}" y_offset="-1"/>
+  <xacro:wheel name="left" side="1" prefix="rear" x_offset="${-wheelbase/2}" y_offset="1"/>
+  <xacro:wheel name="right" side="-1" prefix="rear" x_offset="${-wheelbase/2}" y_offset="-1"/>
+  <!-- 三维激光雷达 -->
+  <link name="lidar">
+    <inertial>
+      <mass value="0.5"/>
+      <inertia>
+        <ixx>0.001</ixx>
+        <iyy>0.001</iyy>
+        <izz>0.001</izz>
+        <ixy>0.0</ixy>
+        <ixz>0.0</ixz>
+        <iyz>0.0</iyz>
+      </inertia>
+    </inertial>
+    <visual>
+      <origin xyz="0 0 0" rpy="0 0 0"/>
+      <geometry>
+        <cylinder radius="${lidar_radius}" length="${lidar_height}"/>
+      </geometry>
+      <material name="silver">
+        <color rgba="0.7 0.7 0.7 1"/>
+      </material>
+    </visual>
+    <collision>
+      <origin xyz="0 0 0" rpy="0 0 0"/>
+      <geometry>
+        <cylinder radius="${lidar_radius}" length="${lidar_height}"/>
+      </geometry>
+    </collision>
+  </link>
+  <joint name="lidar_joint" type="fixed">
+    <parent link="chassis"/>
+    <child link="lidar"/>
+    <origin xyz="0 0 ${chassis_height + lidar_height/2}" rpy="0 0 0"/>
+  </joint>
+  <!-- IMU -->
+  <link name="imu">
+    <inertial>
+      <mass value="0.1"/>
+      <inertia>
+        <ixx>0.0001</ixx>
+        <iyy>0.0001</iyy>
+        <izz>0.0001</izz>
+        <ixy>0.0</ixy>
+        <ixz>0.0</ixz>
+        <iyz>0.0</iyz>
+      </inertia>
+    </inertial>
+    <visual>
+      <origin xyz="0 0 0" rpy="0 0 0"/>
+      <geometry>
+        <box size="${imu_size} ${imu_size} ${imu_size}"/>
+      </geometry>
+      <material name="green">
+        <color rgba="0 1 0 1"/>
+      </material>
+    </visual>
+    <collision>
+      <origin xyz="0 0 0" rpy="0 0 0"/>
+      <geometry>
+        <box size="${imu_size} ${imu_size} ${imu_size}"/>
+      </geometry>
+    </collision>
+  </link>
+  <joint name="imu_joint" type="fixed">
+    <parent link="chassis"/>
+    <child link="imu"/>
+    <origin xyz="0 0 ${chassis_height/2}" rpy="0 0 0"/>
+  </joint>
+  <!-- 摄像头 -->
+  <link name="camera">
+    <inertial>
+      <mass value="0.2"/>
+      <inertia>
+        <ixx>0.0002</ixx>
+        <iyy>0.0002</iyy>
+        <izz>0.0002</izz>
+        <ixy>0.0</ixy>
+        <ixz>0.0</ixz>
+        <iyz>0.0</iyz>
+      </inertia>
+    </inertial>
+    <visual>
+      <origin xyz="0 0 0" rpy="0 0 0"/>
+      <geometry>
+        <box size="${camera_width} ${camera_height} ${camera_depth}"/>
+      </geometry>
+      <material name="red">
+        <color rgba="1 0 0 1"/>
+      </material>
+    </visual>
+    <collision>
+      <origin xyz="0 0 0" rpy="0 0 0"/>
+      <geometry>
+        <box size="${camera_width} ${camera_height} ${camera_depth}"/>
+      </geometry>
+    </collision>
+  </link>
+  <joint name="camera_joint" type="fixed">
+    <parent link="chassis"/>
+    <child link="camera"/>
+    <origin xyz="${chassis_length/2 - 0.1} 0 ${chassis_height}" rpy="0 0 0"/>
+  </joint>
+  <!-- Gazebo 插件 -->
+  <gazebo>
+    <!-- 车身颜色 -->
+    <plugin name="gz_sim_diff_drive" filename="libignition-gazebo-diff-drive-system.so">
+      <left_joint>front_left_wheel_joint</left_joint>
+      <right_joint>front_right_wheel_joint</right_joint>
+      <wheel_separation>${track_width}</wheel_separation>
+      <wheel_radius>${wheel_radius}</wheel_radius>
+      <topic>/cmd_vel</topic>
+      <odom_topic>/odom</odom_topic>
+      <frame_id>odom</frame_id>
+      <child_frame_id>chassis</child_frame_id>
+    </plugin>
+  </gazebo>
+  <!-- LiDAR 传感器 -->
+  <gazebo reference="lidar">
+    <sensor name="lidar_sensor" type="lidar">
+      <pose>0 0 0 0 0 0</pose>
+      <topic>/scan</topic>
+      <update_rate>10</update_rate>
+      <ray>
+        <scan>
+          <horizontal>
+            <samples>360</samples>
+            <resolution>1</resolution>
+            <min_angle>-3.14</min_angle>
+            <max_angle>3.14</max_angle>
+          </horizontal>
+          <vertical>
+            <samples>16</samples>
+            <resolution>1</resolution>
+            <min_angle>-0.26</min_angle>
+            <max_angle>0.26</max_angle>
+          </vertical>
+        </scan>
+        <range>
+          <min>0.1</min>
+          <max>30.0</max>
+          <resolution>0.01</resolution>
+        </range>
+      </ray>
+      <plugin name="gz_sim_lidar" filename="libignition-gazebo-lidar-system.so">
+        <topic>/scan</topic>
+      </plugin>
+    </sensor>
+  </gazebo>
+  <!-- IMU 传感器 -->
+  <gazebo reference="imu">
+    <sensor name="imu_sensor" type="imu">
+      <pose>0 0 0 0 0 0</pose>
+      <topic>/imu/data</topic>
+      <update_rate>100</update_rate>
+      <plugin name="gz_sim_imu" filename="libignition-gazebo-imu-system.so">
+        <topic>/imu/data</topic>
+      </plugin>
+    </sensor>
+  </gazebo>
+  <!-- 摄像头传感器 -->
+  <gazebo reference="camera">
+    <sensor name="camera_sensor" type="camera">
+      <pose>0 0 0 0 0 0</pose>
+      <topic>/camera/image_raw</topic>
+      <update_rate>30</update_rate>
+      <camera>
+        <horizontal_fov>1.57</horizontal_fov>
+        <image>
+          <width>640</width>
+          <height>480</height>
+          <format>R8G8B8</format>
+        </image>
+        <clip>
+          <near>0.1</near>
+          <far>100</far>
+        </clip>
+      </camera>
+      <plugin name="gz_sim_camera" filename="libignition-gazebo-camera-system.so">
+        <topic>/camera/image_raw</topic>
+      </plugin>
+    </sensor>
+  </gazebo>
+  <!-- ROS 2 桥接 -->
+  <gazebo>
+    <plugin name="ros_gz_bridge" filename="libros_gz_bridge.so">
+      <ros>
+        <argument>--ros-args</argument>
+        <argument>-p</argument>
+        <argument>use_sim_time:=true</argument>
+      </ros>
+    </plugin>
+  </gazebo>
 </robot>
+</xacroArtifact>

Commit message: 完全没问题,就差机器人

File: src/ackermann_car/urdf/ackermann_car.xacro (robot description, xacro)
@@ -47,5 +47,5 @@
     </collision>
   </link>
-  <!-- 轮子宏 -->
+  <!-- 轮子宏定义 -->
   <xacro:macro name="wheel" params="name side prefix x_offset y_offset">
     <link name="${prefix}_${name}_wheel">
@@ -98,121 +98,35 @@
   <xacro:wheel name="left" side="1" prefix="rear" x_offset="${-wheelbase/2}" y_offset="1"/>
   <xacro:wheel name="right" side="-1" prefix="rear" x_offset="${-wheelbase/2}" y_offset="-1"/>
-  <!-- 三维激光雷达 -->
+  <!-- LiDAR -->
   <link name="lidar">
-    <inertial>
-      <mass value="0.5"/>
-      <inertia>
-        <ixx>0.001</ixx>
-        <iyy>0.001</iyy>
-        <izz>0.001</izz>
-        <ixy>0.0</ixy>
-        <ixz>0.0</ixz>
-        <iyz>0.0</iyz>
-      </inertia>
-    </inertial>
-    <visual>
-      <origin xyz="0 0 0" rpy="0 0 0"/>
-      <geometry>
-        <cylinder radius="${lidar_radius}" length="${lidar_height}"/>
-      </geometry>
-      <material name="silver">
-        <color rgba="0.7 0.7 0.7 1"/>
-      </material>
-    </visual>
-    <collision>
-      <origin xyz="0 0 0" rpy="0 0 0"/>
-      <geometry>
-        <cylinder radius="${lidar_radius}" length="${lidar_height}"/>
-      </geometry>
-    </collision>
+    <inertial><mass value="0.5"/><inertia><ixx>0.001</ixx><iyy>0.001</iyy><izz>0.001</izz><ixy>0</ixy><ixz>0</ixz><iyz>0</iyz></inertia></inertial>
+    <visual><origin xyz="0 0 0"/><geometry><cylinder radius="${lidar_radius}" length="${lidar_height}"/></geometry></visual>
+    <collision><origin xyz="0 0 0"/><geometry><cylinder radius="${lidar_radius}" length="${lidar_height}"/></geometry></collision>
   </link>
   <joint name="lidar_joint" type="fixed">
-    <parent link="chassis"/>
-    <child link="lidar"/>
+    <parent link="chassis"/><child link="lidar"/>
     <origin xyz="0 0 ${chassis_height + lidar_height/2}" rpy="0 0 0"/>
   </joint>
   <!-- IMU -->
   <link name="imu">
-    <inertial>
-      <mass value="0.1"/>
-      <inertia>
-        <ixx>0.0001</ixx>
-        <iyy>0.0001</iyy>
-        <izz>0.0001</izz>
-        <ixy>0.0</ixy>
-        <ixz>0.0</ixz>
-        <iyz>0.0</iyz>
-      </inertia>
-    </inertial>
-    <visual>
-      <origin xyz="0 0 0" rpy="0 0 0"/>
-      <geometry>
-        <box size="${imu_size} ${imu_size} ${imu_size}"/>
-      </geometry>
-      <material name="green">
-        <color rgba="0 1 0 1"/>
-      </material>
-    </visual>
-    <collision>
-      <origin xyz="0 0 0" rpy="0 0 0"/>
-      <geometry>
-        <box size="${imu_size} ${imu_size} ${imu_size}"/>
-      </geometry>
-    </collision>
+    <inertial><mass value="0.1"/><inertia><ixx>0.0001</ixx><iyy>0.0001</iyy><izz>0.0001</izz><ixy>0</ixy><ixz>0</ixz><iyz>0</iyz></inertia></inertial>
+    <visual><origin xyz="0 0 0"/><geometry><box size="${imu_size} ${imu_size} ${imu_size}"/></geometry></visual>
+    <collision><origin xyz="0 0 0"/><geometry><box size="${imu_size} ${imu_size} ${imu_size}"/></geometry></collision>
   </link>
   <joint name="imu_joint" type="fixed">
-    <parent link="chassis"/>
-    <child link="imu"/>
+    <parent link="chassis"/><child link="imu"/>
     <origin xyz="0 0 ${chassis_height/2}" rpy="0 0 0"/>
   </joint>
   <!-- 摄像头 -->
   <link name="camera">
-    <inertial>
-      <mass value="0.2"/>
-      <inertia>
-        <ixx>0.0002</ixx>
-        <iyy>0.0002</iyy>
-        <izz>0.0002</izz>
-        <ixy>0.0</ixy>
-        <ixz>0.0</ixz>
-        <iyz>0.0</iyz>
-      </inertia>
-    </inertial>
-    <visual>
-      <origin xyz="0 0 0" rpy="0 0 0"/>
-      <geometry>
-        <box size="${camera_width} ${camera_height} ${camera_depth}"/>
-      </geometry>
-      <material name="red">
-        <color rgba="1 0 0 1"/>
-      </material>
-    </visual>
-    <collision>
-      <origin xyz="0 0 0" rpy="0 0 0"/>
-      <geometry>
-        <box size="${camera_width} ${camera_height} ${camera_depth}"/>
-      </geometry>
-    </collision>
+    <inertial><mass value="0.2"/><inertia><ixx>0.0002</ixx><iyy>0.0002</iyy><izz>0.0002</izz><ixy>0</ixy><ixz>0</ixz><iyz>0</iyz></inertia></inertial>
+    <visual><origin xyz="0 0 0"/><geometry><box size="${camera_width} ${camera_height} ${camera_depth}"/></geometry></visual>
+    <collision><origin xyz="0 0 0"/><geometry><box size="${camera_width} ${camera_height} ${camera_depth}"/></geometry></collision>
   </link>
   <joint name="camera_joint" type="fixed">
-    <parent link="chassis"/>
-    <child link="camera"/>
+    <parent link="chassis"/><child link="camera"/>
     <origin xyz="${chassis_length/2 - 0.1} 0 ${chassis_height}" rpy="0 0 0"/>
   </joint>
-  <!-- Gazebo 插件 -->
-  <gazebo>
-    <!-- 车身颜色 -->
-    <plugin name="gz_sim_diff_drive" filename="libignition-gazebo-diff-drive-system.so">
-      <left_joint>front_left_wheel_joint</left_joint>
-      <right_joint>front_right_wheel_joint</right_joint>
-      <wheel_separation>${track_width}</wheel_separation>
-      <wheel_radius>${wheel_radius}</wheel_radius>
-      <topic>/cmd_vel</topic>
-      <odom_topic>/odom</odom_topic>
-      <frame_id>odom</frame_id>
-      <child_frame_id>chassis</child_frame_id>
-    </plugin>
-  </gazebo>
-  <!-- LiDAR 传感器 -->
+  <!-- 插件（仅保留传感器插件） -->
   <gazebo reference="lidar">
     <sensor name="lidar_sensor" type="lidar">
@@ -246,5 +160,4 @@
     </sensor>
   </gazebo>
-  <!-- IMU 传感器 -->
   <gazebo reference="imu">
     <sensor name="imu_sensor" type="imu">
@@ -257,5 +170,4 @@
     </sensor>
   </gazebo>
-  <!-- 摄像头传感器 -->
   <gazebo reference="camera">
     <sensor name="camera_sensor" type="camera">
@@ -280,14 +192,3 @@
     </sensor>
   </gazebo>
-  <!-- ROS 2 桥接 -->
-  <gazebo>
-    <plugin name="ros_gz_bridge" filename="libros_gz_bridge.so">
-      <ros>
-        <argument>--ros-args</argument>
-        <argument>-p</argument>
-        <argument>use_sim_time:=true</argument>
-      </ros>
-    </plugin>
-  </gazebo>
 </robot>
-</xacroArtifact>
